File: homemade-security-key.kicad_pcb (KiCad board)
At the start: 2 copper layers, 22 x 33 mm, 45 parts, among them J1 UP20-C-F-G-FL-1-P12-TR, J2 UP2-AH-1-TH, SW1 SW_Push, U1 AP63203WU-7, U2 W25Q16JVSS, U3 RP2350A-QFN60, Y1 ABM8-272-T3

Commit message: journal and readme done!!
Parts:
- added H1: MountingHole, MountingHole:MountingHole_2.2mm_M2_Pad, F.Cu at (83.5, 83.5)
Routing:
- net GND: vias 141 -> 153
Changed lines of the file:
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@@
 		)
 	)
+	(footprint "MountingHole:MountingHole_2.2mm_M2_Pad"
+		(layer "F.Cu")
+		(at 83.5 83.5)
+		(descr "Mounting Hole 2.2mm, M2, generated by kicad-footprint-generator mountinghole.py")
+		(tags "mountinghole M2")
+		(property "Reference" "H1"
+			(at 0 -3.15 0)
+			(layer "F.SilkS")
+			(effects
+				(font
+					(size 1 1)
+					(thickness 0.15)
+				)
+			)
+		)
+		(property "Value" "MountingHole"
+			(at 0 3.15 0)
+			(layer "F.Fab")
+			(effects
+				(font
+					(size 1 1)
+					(thickness 0.15)
+				)
+			)
+		)
+		(property "Datasheet" ""
+			(at 0 0 0)
+			(layer "F.Fab")
+			(hide yes)
+			(effects
+				(font
+					(size 1.27 1.27)
+					(thickness 0.15)
+				)
+			)
+		)
+		(property "Description" "Mounting Hole without connection"
+			(at 0 0 0)
+			(layer "F.Fab")
+			(hide yes)
+			(effects
+				(font
+					(size 1.27 1.27)
+					(thickness 0.15)
+				)
+			)
+		)
+		(property ki_fp_filters "MountingHole*")
+		(sheetname "/")
+		(sheetfile "homemade-security-key.kicad_sch")
+		(attr exclude_from_pos_files exclude_from_bom)
+		(fp_circle
+			(center 0 0)
+			(end 2.2 0)
+			(stroke
+				(width 0.15)
+				(type solid)
+			)
+			(fill no)
+			(layer "Cmts.User")
+		)
+		(fp_circle
+			(center 0 0)
+			(end 2.45 0)
+			(stroke
+				(width 0.05)
+				(type solid)
+			)
+			(fill no)
+			(layer "F.CrtYd")
+		)
+		(fp_text user "${REFERENCE}"
+			(at 0 0 0)
+			(layer "F.Fab")
+			(effects
+				(font
+					(size 1 1)
+					(thickness 0.15)
+				)
+			)
+		)
+		(pad "1" thru_hole circle
+			(at 0 0)
+			(size 4.4 4.4)
+			(drill 2.2)
+			(layers "*.Cu" "*.Mask")
+			(remove_unused_layers no)
+			(zone_connect 2)
+		)
+		(embedded_fonts no)
+	)
 	(footprint "Capacitor_SMD:C_0402_1005Metric"
 		(layer "F.Cu")
@@
 	)
 	(via
+		(at 83.5 87.25)
+		(size 0.45)
+		(drill 0.225)
+		(layers "F.Cu" "B.Cu")
+		(free yes)
+		(net 2)
+	)
+	(via
+		(at 80.75 86.5)
+		(size 0.45)
+		(drill 0.225)
+		(layers "F.Cu" "B.Cu")
+		(free yes)
+		(net 2)
+	)
+	(via
 		(at 99.76 97.3)
 		(size 0.45)
@@
 	)
 	(via
+		(at 84.75 87)
+		(size 0.45)
+		(drill 0.225)
+		(layers "F.Cu" "B.Cu")
+		(free yes)
+		(net 2)
+	)
+	(via
+		(at 82.75 86.5)
+		(size 0.45)
+		(drill 0.225)
+		(layers "F.Cu" "B.Cu")
+		(free yes)
+		(net 2)
+	)
+	(via
 		(at 98.16 107.5)
 		(size 0.45)
@@
 	)
 	(via
+		(at 85.5 86.25)
+		(size 0.45)
+		(drill 0.225)
+		(layers "F.Cu" "B.Cu")
+		(free yes)
+		(net 2)
+	)
+	(via
 		(at 98.96 84.3)
 		(size 0.45)
@@
 	)
 	(via
+		(at 85.5 87)
+		(size 0.45)
+		(drill 0.225)
+		(layers "F.Cu" "B.Cu")
+		(free yes)
+		(net 2)
+	)
+	(via
 		(at 101.36 97.3)
 		(size 0.45)
@@
 	)
 	(via
+		(at 84.75 86.25)
+		(size 0.45)
+		(drill 0.225)
+		(layers "F.Cu" "B.Cu")
+		(free yes)
+		(net 2)
+	)
+	(via
 		(at 91.76 105.9)
 		(size 0.45)
@@
 	)
 	(via
+		(at 82.75 87.25)
+		(size 0.45)
+		(drill 0.225)
+		(layers "F.Cu" "B.Cu")
+		(free yes)
+		(net 2)
+	)
+	(via
+		(at 83.5 86.5)
+		(size 0.45)
+		(drill 0.225)
+		(layers "F.Cu" "B.Cu")
+		(free yes)
+		(net 2)
+	)
+	(via
 		(at 86.96 82.7)
 		(size 0.45)
@@
 	)
 	(via
+		(at 81.5 85.75)
+		(size 0.45)
+		(drill 0.225)
+		(layers "F.Cu" "B.Cu")
+		(free yes)
+		(net 2)
+	)
+	(via
 		(at 99.76 96.7)
 		(size 0.45)
@@
 	)
 	(via
+		(at 80.75 85.75)
+		(size 0.45)
+		(drill 0.225)
+		(layers "F.Cu" "B.Cu")
+		(free yes)
+		(net 2)
+	)
+	(via
 		(at 91.56 80.5)
 		(size 0.45)
@@
 	)
 	(via
+		(at 81.5 86.5)
+		(size 0.45)
+		(drill 0.225)
+		(layers "F.Cu" "B.Cu")
+		(free yes)
+		(net 2)
+	)
+	(via
 		(at 85.81 103.25)
 		(size 0.45)
@@
 			(pts
 				(xy 92.45 97.25) (xy 94.1 97.25) (xy 94.65 96.7) (xy 94.65 95.7) (xy 94.9 95.45) (xy 96.2 95.45)
-				(xy 96.2175 95.4675) (xy 96.2175 98.03) (xy 92.45 98.03) (xy 92.45 98.03)
+				(xy 96.2175 95.4675) (xy 96.2175 98.03) (xy 92.45 98.03)
 			)
 		)
