File: homemade-security-key.kicad_sch (KiCad schematic)
At the start: 0 parts

Commit message: pcb done!
Parts:
- added C1: 10u, Capacitor_SMD:C_0805_2012Metric, symbol Device:C_Small
- added C10, C11, C14, C2, C4, C5, C6, C7, C8, C9: 100n, Capacitor_SMD:C_0402_1005Metric, symbol Device:C_Small
- added C12: 22u, Capacitor_SMD:C_0603_1608Metric, symbol Device:C_Small
- added C13, C17, C18, C19: 4.7u, Capacitor_SMD:C_0402_1005Metric, symbol Device:C_Small
- added C15, C16: 18p, Capacitor_SMD:C_0402_1005Metric, symbol Device:C_Small
- added C3: 1u, Capacitor_SMD:C_0402_1005Metric, symbol Device:C_Small
- added D1: B38G3RGB-10D0003H2U1930, B38G3RGB_10D0003H2U1930:LED_B38G3RGB-10D0003H2U1930, symbol B38G3RGB-10D0003H2U1930:B38G3RGB-10D0003H2U1930
- added J1: UP20-C-F-G-FL-1-P12-TR, UP20_C_F_G_FL_1_P12_TR:SAMESKY_UP20-C-F-G-FL-1-P12-TR, symbol UP20-C-F-G-FL-1-P12-TR:UP20-C-F-G-FL-1-P12-TR
- added J2: UP2-AH-1-TH, UP2_AH_1_TH:CUI_UP2-AH-1-TH, symbol UP2-AH-1-TH:UP2-AH-1-TH
- added JP1: SolderJumper_2_Bridged, Jumper:SolderJumper-2_P1.3mm_Bridged_RoundedPad1.0x1.5mm, symbol Jumper:SolderJumper_2_Bridged
- added JP2: SolderJumper_2_Open, Jumper:SolderJumper-2_P1.3mm_Open_RoundedPad1.0x1.5mm, symbol Jumper:SolderJumper_2_Open
- added L1: 4.7u, HPC6045NC-4R7M:IND_HPC6045NC_TTA, symbol HPC6045NC-4R7M:HPC6045NC-4R7M
- added L2: AOTA-B201610S3R3-101-T, Inductor_SMD:L_0805_2012Metric_Pad1.15x1.40mm_HandSolder, symbol Device:L
- added R1: 5.1k, Resistor_SMD:R_0402_1005Metric, symbol Device:R
- added R2, R3: 27, Resistor_SMD:R_0402_1005Metric, symbol Device:R_Small
- added R4: 1k, Resistor_SMD:R_0402_1005Metric, symbol Device:R_Small
- added R5: 10k, Resistor_SMD:R_0402_1005Metric, symbol Device:R
- added R6: 147, Resistor_SMD:R_0402_1005Metric, symbol Device:R
- added R7, R8, R9: 33, Resistor_SMD:R_0402_1005Metric, symbol Device:R
- added SW1: SW_Push, PTS526_SM15_SMTR2_LFS:SON4_PTS526 SM15 SMTR2 LFS_CNK, symbol Switch:SW_Push
- added TP1, TP2, TP3, TP4, TP5: TestPoint, TestPoint:TestPoint_Pad_D2.0mm, symbol Connector:TestPoint
- added U1: AP63203WU-7, AP63203WU_7:AP63203WU-7_DIO, symbol AP63203WU_7:AP63203WU-7
- added U2: W25Q16JVSS, Package_SO:SOIC-8_5.3x5.3mm_P1.27mm, symbol Memory_Flash:W25Q16JVSS
- added U3: RP2350A-QFN60, RP2350_KiCad:RP2350A_QFN-60_EP_7.75x7.75_Pitch0.4mm, symbol rp2350a-qfn60:RP2350A-QFN60
- added Y1: ABM8-272-T3, ABM8_272_T3:XTAL_ABM8-272-T3, symbol ABM8-272-T3:ABM8-272-T3
Connections:
- new net: C2.2, L1.2, U1.5 (SW)
- new net: SW1.1, SW1.2, U3.7 (GPIO4)
- new net: R8.1, U3.4 (GPIO2)
- new net: D1.2, R8.2
- new net: R6.1, U3.5 (GPIO3)
- new net: D1.4, R6.2
- new net: C16.2, R4.1, Y1.3
- new net: JP2.2 (B), R5.2, TP1.1, U3.26 (RUN)
- new net: D1.1, R7.2
- new net: TP2.1, U3.40 (GPIO26_ADC0)
- new net: TP4.1, U3.42 (GPIO28_ADC2)
- new net: TP5.1, U3.43 (GPIO29_ADC3)
- new net: J1.A5 (CC1), R1.1
- new net: JP1.2 (B), U1.2 (EN)
- new net: R7.1, U3.3 (GPIO1)
- new net: TP3.1, U3.41 (GPIO27_ADC1)
- new net: C2.1, U1.6 (BST)
- new net +1V1: C19.2, L2.1, U3.23 (DVDD), U3.39 (DVDD), U3.6 (DVDD)
- new net +3.3V: C10.2, C11.2, C12.2, C13.2, C14.2, C17.2, C3.2, C4.2, C5.2, C6.2, C7.2, C8.2, C9.2, D1.3, L1.1, R5.1, R9.1, SW1.3, SW1.4, U1.1 (FB), U2.8 (VCC), U3.1 (IOVDD), U3.11 (IOVDD), U3.20 (IOVDD), U3.30 (IOVDD), U3.38 (IOVDD), U3.44 (ADC_AVDD), U3.45 (IOVDD), U3.49 (VREG_VIN), U3.53 (USB_OTP_VDD), U3.54 (QSPI_IOVDD)
- new net GND: C1.1, C10.1, C11.1, C12.1, C13.1, C14.1, C15.1, C16.1, C17.1, C18.1, C19.1, C3.1, C4.1, C5.1, C6.1, C7.1, C8.1, C9.1, J1.A1 (GND), J1.A12 (GND__1), J1.B12 (GND__2), J1.G1 (SHIELD_GND), J1.G2 (SHIELD_GND__1), J1.G3 (SHIELD_GND__2), J1.G4 (SHIELD_GND__3), J2.4 (GND), J2.SH1 (SHIELD), J2.SH2 (SHIELD__1), JP2.1 (A), R1.2, U1.4 (GND), U2.4 (GND), U3.47 (VREG_PGND), U3.61 (GND), Y1.2 (GND), Y1.4 (GND)
- new net LUSB_D+: R2.2, U3.52 (USB_DP)
- new net LUSB_D-: R3.2, U3.51 (USB_DM)
- new net QSPI_SCLK: U2.6 (CLK), U3.56 (QSPI_SCLK)
- new net QSPI_SD0: U2.5 (DI/IO_{0}), U3.57 (QSPI_SD0)
- new net QSPI_SD1: U2.2 (DO/IO_{1}), U3.59 (QSPI_SD1)
- new net QSPI_SD2: U2.3 (~{WP}/IO_{2}), U3.58 (QSPI_SD2)
- new net QSPI_SD3: U2.7 (~{HOLD}/~{RESET}/IO_{3}), U3.55 (QSPI_SD3)
- new net QSPI_SS: U2.1 (~{CS}), U3.60 (QSPI_SS)
- new net USB_D+: J1.A6 (DP1), J2.3 (D+), R2.1
- new net USB_D-: J1.A7 (DN1), J2.2 (D-), R3.1
- new net VBUS: C1.2, J1.A4 (VBUS), J1.B9 (VBUS__1), J2.1 (VCC), JP1.1 (A), U1.3 (VIN)
- new net VREG_AVDD: C18.2, R9.2, U3.46 (VREG_AVDD)
- new net VREG_LX: L2.2, U3.48 (VREG_LX)
- new net XIN: C15.2, U3.21 (XIN), Y1.1
- new net XOUT: R4.2, U3.22 (XOUT)
Other:
- note added: "3.3V Buck regulator"
- note added: "Crystal"
- note added: "Flash"
- note added: "Onboard regulator"
- note added: "Toby Cm"
- note added: "USB A Plug"
- note added: "USB C Plug"
- note added: "set to LOW to turn LED on"
- title: (none) -> Homemade FIDO Key

Commit message: final push hehe
Parts:
- added H1: MountingHole, MountingHole:MountingHole_2.2mm_M2_Pad, symbol Mechanical:MountingHole
- TP1, TP2, TP3, TP4, TP5: now left out of the parts list
Changed lines of the file:
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@@
 		(unit 1)
 		(exclude_from_sim no)
-		(in_bom yes)
+		(in_bom no)
 		(on_board yes)
 		(dnp no)
@@
 		(unit 1)
 		(exclude_from_sim no)
-		(in_bom yes)
+		(in_bom no)
 		(on_board yes)
 		(dnp no)
@@
 		(unit 1)
 		(exclude_from_sim no)
-		(in_bom yes)
+		(in_bom no)
 		(on_board yes)
 		(dnp no)
@@
 	)
 	(symbol
+		(lib_id "Mechanical:MountingHole")
+		(at 128.27 171.45 0)
+		(unit 1)
+		(exclude_from_sim no)
+		(in_bom no)
+		(on_board yes)
+		(dnp no)
+		(fields_autoplaced yes)
+		(property "Reference" "H1"
+			(at 130.81 169.5449 0)
+			(effects
+				(font
+					(size 1.27 1.27)
+				)
+				(justify left)
+			)
+		)
+		(property "Value" "MountingHole"
+			(at 130.81 173.3549 0)
+			(effects
+				(font
+					(size 1.27 1.27)
+				)
+				(justify left)
+			)
+		)
+		(property "Footprint" "MountingHole:MountingHole_2.2mm_M2_Pad"
+			(at 128.27 171.45 0)
+			(effects
+				(font
+					(size 1.27 1.27)
+				)
+				(hide yes)
+			)
+		)
+		(property "Datasheet" "~"
+			(at 128.27 171.45 0)
+			(effects
+				(font
+					(size 1.27 1.27)
+				)
+				(hide yes)
+			)
+		)
+		(property "Description" "Mounting Hole without connection"
+			(at 128.27 171.45 0)
+			(effects
+				(font
+					(size 1.27 1.27)
+				)
+				(hide yes)
+			)
+		)
+		(instances
+			(project ""
+				(path "/e348423a-8fc2-43e1-bc35-c9787ab22481"
+					(reference "H1")
+					(unit 1)
+				)
+			)
+		)
+	)
+	(symbol
 		(lib_id "Device:C_Small")
 		(at 158.75 34.29 0)
@@
 		(unit 1)
 		(exclude_from_sim no)
-		(in_bom yes)
+		(in_bom no)
 		(on_board yes)
 		(dnp no)
@@
 		(unit 1)
 		(exclude_from_sim no)
-		(in_bom yes)
+		(in_bom no)
 		(on_board yes)
 		(dnp no)
